File: KiCAD/VideoCounter.kicad_sch (KiCad schematic)
At the start: 11 parts

Commit message: Update schematics
- Bugfixes for addressing
- Adding more info on PAL in video circuit
Other:
- note added: "1.32 kHz (1.30 kHz)"
- note added: "165 Hz (162.5 Hz)"
- note added: "330 Hz (325 Hz)"
- note added: "60 Hz (50 Hz)"
- note added: "660 Hz (650 Hz)"
- note added: "82.5 Hz (81.25 Hz)"
- note added: "CP0/11 (CP0/13)"
- note added: "CP0/12 (CP0/12 or 13)"
- note added: "NTSC"
- note added: "NTSC (PAL)"
- note added: "PAL"
- note removed: "1.32 kHz"
- note removed: "165 Hz"
- note removed: "330 Hz"
- note removed: "60 Hz"
- note removed: "660 Hz"
- note removed: "82.5 Hz"
- note removed: "CP0/11"
- note removed: "CP0/12"
- moved on the sheet: JP6
