File: KiCAD/VideoSync.kicad_sch (KiCad schematic)
At the start: 9 parts

Commit message: Update schematics
- Bugfixes for addressing
- Adding more info on PAL in video circuit
Changed lines of the file:
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@@
 	(title_block
 		(title "TRS-80 Model I Rev HE11E011520")
-		(date "2025-06-14")
+		(date "2025-06-15")
 		(rev "E1A")
 		(company "RetroStack - Marcel Erz")
@@
 		(stroke
 			(width 0)
+			(type default)
+		)
+	)
+	(bus_entry
+		(at 161.925 111.125)
+		(size 2.54 2.54)
+		(stroke
+			(width 0)
